Commit message: Updated core URDF - added material colors

File: description/robot_core.xacro (robot description, xacro)
@@ -29,4 +29,5 @@
 				<box size="0.3 0.3 0.15" />
 			</geometry>
+			<material name="white" />
 		</visual>
 		<collision>
@@ -52,4 +53,5 @@
 				<cylinder radius="0.05" length="0.04" />
 			</geometry>
+			<material name="white" />
 		</visual>
 		<collision>
@@ -74,4 +76,5 @@
 				<cylinder radius="0.05" length="0.04" />
 			</geometry>
+			<material name="white" />
 		</visual>
 		<collision>
@@ -95,4 +98,5 @@
 				<sphere radius="0.05" />
 			</geometry>
+			<material name="black" />
 		</visual>
 		<collision>
