Commit message: changed depth and core parameters, also shifting to linux

File: description/depth_camera.xacro (robot description, xacro)
@@ -25,5 +25,5 @@
         <sensor name="camera" type="depth">
             <pose>0 0 0 0 0 0</pose>
-            <visualize>true</visualize>
+            <visualize>false</visualize>
             <update_rate>10</update_rate>
             <camera>

File: description/robot_core.xacro (robot description, xacro)
@@ -21,4 +21,12 @@
 	<link name="base_link">
 	</link>
+	<!-- BASE_FOOTPRINT-->
+	 <joint name="base_footprint_joint" type="fixed">
+		<parent link="base_link"/>
+		<child link="base_footprint"/>
+		<origin xyz="0 0 0" rpy="0 0 0"/>
+	 </joint>
+	 <link name="base_footprint">
+	 </link>
 	<!-- CHASSIS LINK -->
 	<joint name="chassis_joint" type="fixed">
